File: pcb/intertubeClock.brd (EAGLE design)
At the start: 166.3 x 53.8 mm, 174 parts, among them Q1 TP5322K1-G, Q10 TP5322K1-G, Q11 TP5322K1-G, Q12 TP5322K1-G, Q13 TP5322K1-G, Q14 TP5322K1-G, Q15 TP5322K1-G, Q16 TP5322K1-G, Q17 NX138AK, Q18 NX138AK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

Commit message: -Completed layout.
Parts:
- added JP14: (no value), pinhead:2X04
- JP10: device pinhead:1X06 -> pinhead:1X07
- moved C3 4.50 mm to (115.1, 36.3), turned to 180 degrees
- moved R1 2.30 mm to (149.1, 41.1)
- moved R2 2.30 mm to (153.2, 41.1)
- moved R4 2.30 mm to (136.9, 41.1)
- moved JP2 2.30 mm to (158.0, 41.1), turned to 180 degrees
- moved R3 2.30 mm to (141.0, 41.1)
- moved R5 2.30 mm to (145.0, 41.1)
- moved C4 2.18 mm to (115.1, 38.9), turned to 180 degrees
- moved JP13 1.85 mm to (153.2, 47.2), turned to 0 degrees
- moved JP12 1.80 mm to (145.0, 47.2), turned to 0 degrees
- moved JP11 1.78 mm to (136.9, 47.2), turned to 0 degrees
- moved JP10 1.27 mm to (12.4, 47.2), turned to 0 degrees
- moved Q17 0.51 mm to (19.8, 39.9)
- moved R118 0.51 mm to (19.8, 43.2)
- moved R122 0.51 mm to (19.8, 36.8)
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Connections:
- new net SPARE1: JP14.1, U2.16
- new net SPARE2: JP14.2, U2.17
- new net SPARE3: JP14.3, U2.18
- new net SPARE4: JP14.4, U2.19
- new net SPARE5: JP14.5, U2.20
- new net SPARE6: JP14.6, U2.21
- new net SPARE7: JP14.7, U2.22
- net CLK: now also JP10.6; no longer JP10.3, U2.29
- net CLK_HV: now also U2.29
- net DATA_IN: now also JP10.7; no longer JP10.2
- net GND: now also JP10.3; no longer JP10.1
- net OE: now also JP10.5; no longer JP10.4, U2.28
- net OE_HV: now also U2.28
- net STR: now also JP10.4; no longer JP10.5, U2.32
- net STR_HV: now also U2.32
- net VCC: now also JP10.2
- net VDD: now also JP10.1; no longer JP10.6
Routing:
- net HV_VS: track 0.00 -> 206.5 mm, vias 0 -> 15
- net VCC: track 0.00 -> 138.9 mm, vias 0 -> 6
- net DATA_OUT2_HV: track 0.00 -> 120.5 mm, vias 0 -> 2
- net STR_HV: track 0.00 -> 116.2 mm, vias 0 -> 3
- net OE_HV: track 0.00 -> 113.9 mm, vias 0 -> 3
- net CLK_HV: track 0.00 -> 110.8 mm, vias 0 -> 3
- net DATA_OUT1_HV: track 0.00 -> 69.0 mm
- net K89_DIG8: track 0.00 -> 58.3 mm, vias 0 -> 3
- net K01_DIG8: track 6.22 -> 63.3 mm, vias 1 -> 3
- net K45_DIG8: track 0.00 -> 56.0 mm, vias 0 -> 3
- net K67_DIG8: track 0.00 -> 55.7 mm, vias 0 -> 3
- net K23_DIG8: track 0.00 -> 54.6 mm, vias 0 -> 3
- net A2_SEL#_DIG5: track 0.00 -> 45.4 mm
- net A1_SEL#_DIG5: track 0.00 -> 37.8 mm
- net DATA_IN_HV: track 0.00 -> 26.0 mm, vias 0 -> 2
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