File: pcb/intertubeClock.sch (EAGLE design)
At the start: 174 parts, among them Q1 TP5322K1-G, Q10 TP5322K1-G, Q11 TP5322K1-G, Q12 TP5322K1-G, Q13 TP5322K1-G, Q14 TP5322K1-G, Q15 TP5322K1-G, Q16 TP5322K1-G, Q17 NX138AK, Q18 NX138AK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

Commit message: -Completed layout.
Parts:
- added JP14: (no value), pinhead:PINHD-2X4
- JP10: device pinhead:PINHD-1X6 -> pinhead:PINHD-1X7
Connections:
- new net SPARE1: JP14.1, U2.HVOUT26
- new net SPARE2: JP14.2, U2.HVOUT27
- new net SPARE3: JP14.3, U2.HVOUT28
- new net SPARE4: JP14.4, U2.HVOUT29
- new net SPARE5: JP14.5, U2.HVOUT30
- new net SPARE6: JP14.6, U2.HVOUT31
- new net SPARE7: JP14.7, U2.HVOUT32
- net CLK: now also JP10.6; no longer JP10.3, U2.CLK
- net CLK_HV: now also U2.CLK
- net DATA_IN: now also JP10.7; no longer JP10.2
- net GND: now also JP10.3; no longer JP10.1
- net OE: now also JP10.5; no longer JP10.4, U2.OE
- net OE_HV: now also U2.OE
- net STR: now also JP10.4; no longer JP10.5, U2.STR
- net STR_HV: now also U2.STR
- net VCC: now also JP10.2
- net VDD: now also JP10.1; no longer JP10.6
Other:
- note added: "2019.05.19"
- note added: "COMPLETED LAYOUT"
Changed lines of the file:
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@@
 <part name="R125" library="rcl" deviceset="R-US_" device="R0603" value="10K"/>
 <part name="P+3" library="supply1" deviceset="VCC" device=""/>
-<part name="JP10" library="pinhead" deviceset="PINHD-1X6" device=""/>
 <part name="R126" library="rcl" deviceset="R-US_" device="R0603" value="10K"/>
 <part name="GND10" library="supply1" deviceset="GND" device=""/>
@@
 <part name="Q7" library="intertubeClock" deviceset="TP5322" device="K1-G"/>
 <part name="Q8" library="intertubeClock" deviceset="TP5322" device="K1-G"/>
+<part name="JP10" library="pinhead" deviceset="PINHD-1X7" device=""/>
+<part name="JP14" library="pinhead" deviceset="PINHD-2X4" device=""/>
 </parts>
 <sheets>
@@
 <text x="193.04" y="165.1" size="2.54" layer="94" rot="MR180">CONTINUED LAYOUT
 PINSWAPPED DIODES</text>
+<text x="50.8" y="152.4" size="2.54" layer="94">ANDERS NELSON</text>
+<text x="144.78" y="152.4" size="2.54" layer="94">2019.05.19</text>
+<text x="193.04" y="154.94" size="2.54" layer="94" rot="MR180">COMPLETED LAYOUT</text>
 </plain>
 <instances>
@@
 <attribute name="VALUE" x="193.04" y="152.4" size="1.778" layer="96" rot="R180"/>
 </instance>
-<instance part="JP10" gate="A" x="25.4" y="121.92" rot="MR0"/>
 <instance part="R126" gate="G$1" x="142.24" y="48.26" smashed="yes" rot="MR270">
 <attribute name="NAME" x="139.7" y="40.64" size="1.778" layer="95" rot="MR90"/>
@@
 <instance part="Q20" gate="G$1" x="78.74" y="40.64"/>
 <instance part="Q21" gate="G$1" x="144.78" y="33.02" rot="MR0"/>
+<instance part="JP10" gate="A" x="25.4" y="119.38" smashed="yes" rot="R180">
+<attribute name="NAME" x="24.13" y="130.175" size="1.778" layer="95"/>
+<attribute name="VALUE" x="31.75" y="132.08" size="1.778" layer="96" rot="R180"/>
+</instance>
+<instance part="JP14" gate="A" x="335.28" y="66.04"/>
 </instances>
 <busses>
@@
 </segment>
 <segment>
-<wire x1="27.94" y1="129.54" x2="48.26" y2="129.54" width="0.1524" layer="91"/>
-<label x="35.56" y="129.54" size="1.778" layer="95"/>
-<pinref part="JP10" gate="A" pin="1"/>
+<wire x1="27.94" y1="116.84" x2="48.26" y2="116.84" width="0.1524" layer="91"/>
+<label x="35.56" y="116.84" size="1.778" layer="95"/>
+<pinref part="JP10" gate="A" pin="3"/>
 </segment>
 <segment>
@@
 <junction x="58.42" y="119.38"/>
 <wire x1="58.42" y1="127" x2="58.42" y2="119.38" width="0.1524" layer="91"/>
-<pinref part="JP10" gate="A" pin="2"/>
 <pinref part="Q17" gate="G$1" pin="G"/>
+<pinref part="JP10" gate="A" pin="7"/>
 </segment>
 </net>
@@
 <wire x1="58.42" y1="86.36" x2="58.42" y2="91.44" width="0.1524" layer="91"/>
 <junction x="58.42" y="91.44"/>
-<pinref part="JP10" gate="A" pin="3"/>
 <pinref part="Q18" gate="G$1" pin="G"/>
-</segment>
-<segment>
-<pinref part="U2" gate="G$1" pin="CLK"/>
-<wire x1="215.9" y1="134.62" x2="241.3" y2="134.62" width="0.1524" layer="91"/>
-<label x="218.44" y="134.62" size="1.778" layer="95"/>
+<pinref part="JP10" gate="A" pin="6"/>
 </segment>
 </net>
@@
 <junction x="58.42" y="63.5"/>
 <wire x1="53.34" y1="63.5" x2="58.42" y2="63.5" width="0.1524" layer="91"/>
-<pinref part="JP10" gate="A" pin="4"/>
 <pinref part="Q19" gate="G$1" pin="G"/>
-</segment>
-<segment>
-<pinref part="U2" gate="G$1" pin="OE"/>
-<wire x1="241.3" y1="129.54" x2="215.9" y2="129.54" width="0.1524" layer="91"/>
-<label x="218.44" y="129.54" size="1.778" layer="95"/>
+<pinref part="JP10" gate="A" pin="5"/>
 </segment>
 </net>
@@
 <junction x="58.42" y="38.1"/>
 <wire x1="50.8" y1="38.1" x2="58.42" y2="38.1" width="0.1524" layer="91"/>
-<pinref part="JP10" gate="A" pin="5"/>
 <pinref part="Q20" gate="G$1" pin="G"/>
-</segment>
-<segment>
-<pinref part="U2" gate="G$1" pin="STR"/>
-<wire x1="215.9" y1="127" x2="241.3" y2="127" width="0.1524" layer="91"/>
-<label x="218.44" y="127" size="1.778" layer="95"/>
+<pinref part="JP10" gate="A" pin="4"/>
 </segment>
 </net>
@@
 <net name="SPARE1" class="0">
 <segment>
-<wire x1="294.64" y1="76.2" x2="314.96" y2="76.2" width="0.1524" layer="91"/>
-<label x="297.18" y="76.2" size="1.778" layer="95"/>
+<wire x1="274.32" y1="76.2" x2="294.64" y2="76.2" width="0.1524" layer="91"/>
+<label x="276.86" y="76.2" size="1.778" layer="95"/>
+<pinref part="U2" gate="G$1" pin="HVOUT26"/>
+</segment>
+<segment>
+<wire x1="312.42" y1="71.12" x2="332.74" y2="71.12" width="0.1524" layer="91"/>
+<label x="314.96" y="71.12" size="1.778" layer="95"/>
+<pinref part="JP14" gate="A" pin="1"/>
 </segment>
 </net>
 <net name="SPARE2" class="0">
 <segment>
-<wire x1="294.64" y1="73.66" x2="314.96" y2="73.66" width="0.1524" layer="91"/>
-<label x="297.18" y="73.66" size="1.778" layer="95"/>
+<wire x1="274.32" y1="73.66" x2="294.64" y2="73.66" width="0.1524" layer="91"/>
+<label x="276.86" y="73.66" size="1.778" layer="95"/>
+<pinref part="U2" gate="G$1" pin="HVOUT27"/>
+</segment>
+<segment>
+<wire x1="340.36" y1="71.12" x2="360.68" y2="71.12" width="0.1524" layer="91"/>
+<label x="342.9" y="71.12" size="1.778" layer="95"/>
+<pinref part="JP14" gate="A" pin="2"/>
 </segment>
 </net>
 <net name="SPARE3" class="0">
 <segment>
-<wire x1="294.64" y1="71.12" x2="314.96" y2="71.12" width="0.1524" layer="91"/>
-<label x="297.18" y="71.12" size="1.778" layer="95"/>
+<wire x1="274.32" y1="71.12" x2="294.64" y2="71.12" width="0.1524" layer="91"/>
+<label x="276.86" y="71.12" size="1.778" layer="95"/>
+<pinref part="U2" gate="G$1" pin="HVOUT28"/>
+</segment>
+<segment>
+<wire x1="312.42" y1="68.58" x2="332.74" y2="68.58" width="0.1524" layer="91"/>
+<label x="314.96" y="68.58" size="1.778" layer="95"/>
+<pinref part="JP14" gate="A" pin="3"/>
 </segment>
 </net>
 <net name="SPARE4" class="0">
 <segment>
-<wire x1="294.64" y1="68.58" x2="314.96" y2="68.58" width="0.1524" layer="91"/>
-<label x="297.18" y="68.58" size="1.778" layer="95"/>
+<wire x1="274.32" y1="68.58" x2="294.64" y2="68.58" width="0.1524" layer="91"/>
+<label x="276.86" y="68.58" size="1.778" layer="95"/>
+<pinref part="U2" gate="G$1" pin="HVOUT29"/>
+</segment>
+<segment>
+<wire x1="340.36" y1="68.58" x2="360.68" y2="68.58" width="0.1524" layer="91"/>
+<label x="342.9" y="68.58" size="1.778" layer="95"/>
+<pinref part="JP14" gate="A" pin="4"/>
 </segment>
 </net>
 <net name="SPARE5" class="0">
 <segment>
-<wire x1="294.64" y1="66.04" x2="314.96" y2="66.04" width="0.1524" layer="91"/>
-<label x="297.18" y="66.04" size="1.778" layer="95"/>
+<wire x1="274.32" y1="66.04" x2="294.64" y2="66.04" width="0.1524" layer="91"/>
+<label x="276.86" y="66.04" size="1.778" layer="95"/>
+<pinref part="U2" gate="G$1" pin="HVOUT30"/>
+</segment>
+<segment>
+<wire x1="312.42" y1="66.04" x2="332.74" y2="66.04" width="0.1524" layer="91"/>
+<label x="314.96" y="66.04" size="1.778" layer="95"/>
+<pinref part="JP14" gate="A" pin="5"/>
 </segment>
 </net>
 <net name="SPARE6" class="0">
 <segment>
-<wire x1="294.64" y1="63.5" x2="314.96" y2="63.5" width="0.1524" layer="91"/>
-<label x="297.18" y="63.5" size="1.778" layer="95"/>
+<wire x1="274.32" y1="63.5" x2="294.64" y2="63.5" width="0.1524" layer="91"/>
+<label x="276.86" y="63.5" size="1.778" layer="95"/>
+<pinref part="U2" gate="G$1" pin="HVOUT31"/>
+</segment>
+<segment>
+<wire x1="340.36" y1="66.04" x2="360.68" y2="66.04" width="0.1524" layer="91"/>
+<label x="342.9" y="66.04" size="1.778" layer="95"/>
+<pinref part="JP14" gate="A" pin="6"/>
 </segment>
 </net>
 <net name="SPARE7" class="0">
 <segment>
-<wire x1="294.64" y1="60.96" x2="314.96" y2="60.96" width="0.1524" layer="91"/>
-<label x="297.18" y="60.96" size="1.778" layer="95"/>
+<wire x1="274.32" y1="60.96" x2="294.64" y2="60.96" width="0.1524" layer="91"/>
+<label x="276.86" y="60.96" size="1.778" layer="95"/>
+<pinref part="U2" gate="G$1" pin="HVOUT32"/>
+</segment>
+<segment>
+<wire x1="312.42" y1="63.5" x2="332.74" y2="63.5" width="0.1524" layer="91"/>
+<label x="314.96" y="63.5" size="1.778" layer="95"/>
+<pinref part="JP14" gate="A" pin="7"/>
 </segment>
 </net>
@@
 <label x="223.52" y="236.22" size="1.778" layer="95"/>
 </segment>
+<segment>
+<wire x1="215.9" y1="134.62" x2="241.3" y2="134.62" width="0.1524" layer="91"/>
+<label x="218.44" y="134.62" size="1.778" layer="95"/>
+<pinref part="U2" gate="G$1" pin="CLK"/>
+</segment>
 </net>
 <net name="OE_HV" class="0">
@@
 <label x="223.52" y="231.14" size="1.778" layer="95"/>
 </segment>
+<segment>
+<wire x1="241.3" y1="129.54" x2="215.9" y2="129.54" width="0.1524" layer="91"/>
+<label x="218.44" y="129.54" size="1.778" layer="95"/>
+<pinref part="U2" gate="G$1" pin="OE"/>
+</segment>
 </net>
 <net name="STR_HV" class="0">
@@
 <wire x1="220.98" y1="228.6" x2="241.3" y2="228.6" width="0.1524" layer="91"/>
 <label x="223.52" y="228.6" size="1.778" layer="95"/>
+</segment>
+<segment>
+<wire x1="215.9" y1="127" x2="241.3" y2="127" width="0.1524" layer="91"/>
+<label x="218.44" y="127" size="1.778" layer="95"/>
+<pinref part="U2" gate="G$1" pin="STR"/>
 </segment>
 </net>
@@
 <pinref part="P+1" gate="VCC" pin="VCC"/>
 </segment>
+<segment>
+<wire x1="27.94" y1="114.3" x2="48.26" y2="114.3" width="0.1524" layer="91"/>
+<label x="35.56" y="114.3" size="1.778" layer="95"/>
+<pinref part="JP10" gate="A" pin="2"/>
+</segment>
 </net>
 <net name="VDD" class="0">
 <segment>
-<pinref part="JP10" gate="A" pin="6"/>
-<wire x1="27.94" y1="116.84" x2="48.26" y2="116.84" width="0.1524" layer="91"/>
-<label x="35.56" y="116.84" size="1.778" layer="95"/>
-</segment>
-<segment>
+<wire x1="27.94" y1="111.76" x2="48.26" y2="111.76" width="0.1524" layer="91"/>
+<label x="35.56" y="111.76" size="1.778" layer="95"/>
+<pinref part="JP10" gate="A" pin="1"/>
+</segment>
+<segment>
